Commit message: updated mass and bounding box

File: urdf/custom_jackal.urdf.xacro (robot description, xacro)
@@ -4,5 +4,5 @@
     <link name="right_tag">
         <inertial>
-            <mass value="1" />
+            <mass value="0.1" />
             <inertia ixx="1.0" ixy="0.0" ixz="0.0" iyy="1.0" iyz="0.0" izz="1.0" />
         </inertial>
@@ -10,5 +10,5 @@
             <origin xyz="0 0 0" rpy="0 0 0"/>
             <geometry>
-                <box size="0.01 0.01 0.01"/>
+                <box size="0.05 0.026 0.102"/>
             </geometry>
         </collision>
@@ -31,5 +31,5 @@
     <link name="left_tag">
         <inertial>
-            <mass value="1" />
+            <mass value="0.1" />
             <inertia ixx="1.0" ixy="0.0" ixz="0.0" iyy="1.0" iyz="0.0" izz="1.0" />
         </inertial>
@@ -37,5 +37,5 @@
             <origin xyz="0 0 0" rpy="0 0 0"/>
             <geometry>
-                <box size="0.01 0.01 0.01"/>
+                <box size="0.05 0.026 0.102"/>
             </geometry>
         </collision>

Commit message: fixed tags not being seen by gazebo plugin
this is due to the fixed joints being removed by the sdf conversion.

Needed to add the preserve fixed joint tag and also have the joints linked to the base link

File: urdf/custom_jackal.urdf.xacro (robot description, xacro)
@@ -5,4 +5,5 @@
         <inertial>
             <mass value="0.1" />
+            <origin rpy="0 0 0" xyz="0 0 0"/>
             <inertia ixx="1.0" ixy="0.0" ixz="0.0" iyy="1.0" iyz="0.0" izz="1.0" />
         </inertial>
@@ -21,9 +22,12 @@
     </link>
     <joint name="right_tag_joint" type="fixed">
-        <!-- <origin xyz="0.161786 0 0.2378375000000002" rpy="0 0 0"/> -->
-        <origin xyz="0 0.161786 0" rpy="0 0 3.14159265359"/>
-        <parent link="mid_mount"/>
+        <origin xyz="0 0.161786 0.184" rpy="0 0 3.14159265359"/>
+        <!-- <origin xyz="0 0.161786 0" rpy="0 0 3.14159265359"/> -->
+        <parent link="base_link"/>
         <child link="right_tag"/>
-     </joint>
+    </joint>
+    <gazebo reference="right_tag_joint">
+        <preserveFixedJoint>true</preserveFixedJoint>
+    </gazebo>
     <gazebo reference="right_tag">
         <material>Gazebo/White</material>
@@ -32,4 +36,5 @@
         <inertial>
             <mass value="0.1" />
+            <origin rpy="0 0 0" xyz="0 0 0"/>
             <inertia ixx="1.0" ixy="0.0" ixz="0.0" iyy="1.0" iyz="0.0" izz="1.0" />
         </inertial>
@@ -48,9 +53,12 @@
     </link>
     <joint name="left_tag_joint" type="fixed">
-        <!-- <origin xyz="0.161786 0 0.2378375000000002" rpy="0 0 0"/> -->
-        <origin xyz="0 -0.161786 0" rpy="0 0 0"/>
-        <parent link="mid_mount"/>
+        <origin xyz="0 -0.161786 0.184" rpy="0 0 0"/>
+        <!-- <origin xyz="0 -0.161786 0" rpy="0 0 0"/> -->
+        <parent link="base_link"/>
         <child link="left_tag"/>
-     </joint>
+    </joint>
+    <gazebo reference="left_tag_joint">
+        <preserveFixedJoint>true</preserveFixedJoint>
+    </gazebo>
     <gazebo reference="left_tag">
         <material>Gazebo/White</material>

Commit message: fixed collision box location

File: urdf/custom_jackal.urdf.xacro (robot description, xacro)
@@ -9,5 +9,5 @@
         </inertial>
         <collision>
-            <origin xyz="0 0 0" rpy="0 0 0"/>
+            <origin xyz="0 -0.013 0" rpy="0 0 0"/>
             <geometry>
                 <box size="0.05 0.026 0.102"/>
@@ -40,5 +40,5 @@
         </inertial>
         <collision>
-            <origin xyz="0 0 0" rpy="0 0 0"/>
+            <origin xyz="0 -0.013 0" rpy="0 0 0"/>
             <geometry>
                 <box size="0.05 0.026 0.102"/>

Commit message: fixed jackal tag labeling

File: urdf/custom_jackal.urdf.xacro (robot description, xacro)
@@ -22,5 +22,5 @@
     </link>
     <joint name="right_tag_joint" type="fixed">
-        <origin xyz="0 0.161786 0.184" rpy="0 0 3.14159265359"/>
+        <origin xyz="0 -0.161786 0.184" rpy="0 0 0"/>
         <!-- <origin xyz="0 0.161786 0" rpy="0 0 3.14159265359"/> -->
         <parent link="base_link"/>
@@ -53,5 +53,5 @@
     </link>
     <joint name="left_tag_joint" type="fixed">
-        <origin xyz="0 -0.161786 0.184" rpy="0 0 0"/>
+        <origin xyz="0 0.161786 0.184" rpy="0 0 3.14159265359"/>
         <!-- <origin xyz="0 -0.161786 0" rpy="0 0 0"/> -->
         <parent link="base_link"/>

Commit message: added the ability to specify Jacakal tag number from roslaunch

File: urdf/custom_jackal.urdf.xacro (robot description, xacro)
@@ -2,4 +2,8 @@
 <robot xmlns:xacro="http://www.ros.org/wiki/xacro" name="Jackal">
     <xacro:include filename="$(find jackal_description)/urdf/jackal.urdf.xacro" />
+    <xacro:arg name="right_id" default="0" />
+    <xacro:arg name="left_id" default="1" />
+    <xacro:property name="right" value="$(arg right_id)" />
+    <xacro:property name="left" value="$(arg left_id)" />
     <link name="right_tag">
         <inertial>
@@ -72,5 +76,5 @@
             <tag_link>right_tag</tag_link>
             <anchor_prefix>uwb_anchor</anchor_prefix>
-            <tag_id>0</tag_id>
+            <tag_id>${right}</tag_id>
             <noise type='gaussian'>
                 <mean>0</mean>
@@ -87,5 +91,5 @@
             <tag_link>left_tag</tag_link>
             <anchor_prefix>uwb_anchor</anchor_prefix>
-            <tag_id>1</tag_id>
+            <tag_id>${left}</tag_id>
             <noise type='gaussian'>
                 <mean>0</mean>
