Commit message: Added ability to specifigy the anchor number in roslaunch

File: urdf/custom_anchor_jackal.urdf.xacro (robot description, xacro)
@@ -1,6 +1,8 @@
 <?xml version="1.0"?>
 <robot xmlns:xacro="http://www.ros.org/wiki/xacro" name="Jackal">
+    <xacro:arg name="anchor_id" default="-1" />
+    <xacro:property name="anchor" value="$(arg anchor_id)" />
     <xacro:include filename="$(find jackal_world)/urdf/custom_jackal.urdf.xacro" />
-    <link name="uwb_anchor10">
+    <link name="uwb_anchor${anchor}">
         <inertial>
             <mass value="0.1" />
@@ -24,10 +26,10 @@
         <origin xyz="0 0 0.25" rpy="0 0 1.57079632679"/>
         <parent link="base_link"/>
-        <child link="uwb_anchor10"/>
+        <child link="uwb_anchor${anchor}"/>
     </joint>
     <gazebo reference="uwb_anchor_joint">
         <preserveFixedJoint>true</preserveFixedJoint>
     </gazebo>
-    <gazebo reference="uwb_anchor10">
+    <gazebo reference="uwb_anchor${anchor}">
         <material>Gazebo/White</material>
     </gazebo>
