Commit message: added namespace parameter to drone URDF

File: urdf/custom_sjtu_drone.urdf.xacro (robot description, xacro)
@@ -1,6 +1,8 @@
 <?xml version="1.0" ?>
 <robot xmlns:xacro="http://www.ros.org/wiki/xacro" name="sjut_drone">
-      <xacro:arg name="anchor_id" default="-1" />
-    <xacro:property name="anchor" value="$(arg anchor_id)" />
+  <xacro:arg name="anchor_id" default="-1" />
+  <xacro:property name="anchor" value="$(arg anchor_id)" />
+  <xacro:arg name="ns" default="/" />
+  <xacro:property name="ns" value="$(arg ns)"/>
   <link name="base_link">
     <inertial>
@@ -26,4 +28,5 @@
         <bodyName>base_link</bodyName>
         <imuTopic>/drone/imu</imuTopic>
+        <robotNamespace>${ns}</robotNamespace>
         <rollpitchProportionalGain>10.0</rollpitchProportionalGain>
         <rollpitchDifferentialGain>5.0</rollpitchDifferentialGain>
@@ -82,7 +85,9 @@
   </gazebo>
   <!-- Sensors -->
-  <!-- <gazebo>
+  <gazebo>
     	<sensor name='sensor_imu' type='imu'>
         <always_on> 1 </always_on>
+        <robotNamespace>${ns}</robotNamespace>
+        <topicName>drone/imu</topicName>
         <update_rate> 100 </update_rate>
         <pose> 0 0 0 0 0 0 </pose>
@@ -102,5 +107,6 @@
           </noise>
         </imu>
-      </sensor> -->
+      </sensor>
+    </gazebo>
       <!-- Sonar sensor in 100fps -->
       <!-- <sensor name='sensor_sonar' type='sonar'>
